Commit message: urdfs all setup, need to implement controls

File: urdf/umbc_husky.urdf.xacro (robot description, xacro)
@@ -21,9 +21,9 @@
 ARISING IN ANY WAY OUT OF THE USE OF THIS SOFTWARE, EVEN IF ADVISED OF THE POSSIBILITY OF SUCH DAMAGE.
 -->
-<robot name="husky" xmlns:xacro="http://ros.org/wiki/xacro">
+<robot name="husky" xmlns:xacro="http://www.ros.org/wiki/xacro">
   <xacro:arg name="laser_enabled" default="false" />
   <xacro:arg name="laser_xyz" default="$(optenv HUSKY_LMS1XX_XYZ 0.2206 0.0 0.00635)" />
   <xacro:arg name="laser_rpy" default="$(optenv HUSKY_LMS1XX_RPY 0.0 0.0 0.0)" />
-  <xacro:arg name="kinect_enabled" default="false" />
+  <xacro:arg name="kinect_enabled" default="true" />
   <xacro:arg name="kinect_xyz" default="$(optenv HUSKY_KINECT_XYZ 0 0 0)" />
   <xacro:arg name="kinect_rpy" default="$(optenv HUSKY_KINECT_RPY 0 0.18 3.14)" />
@@ -31,5 +31,5 @@
   <xacro:property name="husky_rear_bumper_extend" value="$(optenv HUSKY_REAR_BUMPER_EXTEND 0)" />
   <xacro:arg name="robot_namespace" default="/" />
-  <xacro:arg name="urdf_extras" default="empty.urdf" />
+  <xacro:arg name="urdf_extras" default="$(find husky_description)/urdf/empty.urdf" />
   <!-- Included URDF/XACRO Files -->
   <xacro:include filename="$(find husky_description)/urdf/decorations.urdf.xacro" />
@@ -115,13 +115,4 @@
   </xacro:husky_wheel>
   <xacro:husky_decorate />
-  <xacro:if value="$(arg laser_enabled)">
-    <sick_lms1xx_mount prefix="base"/>
-    <sick_lms1xx frame="base_laser" topic="scan" robot_namespace="$(arg robot_namespace)"/>
-    <joint name="laser_mount_joint" type="fixed">
-      <origin xyz="$(arg laser_xyz)" rpy="$(arg laser_rpy)" />
-      <parent link="top_plate_link" />
-      <child link="base_laser_mount" />
-    </joint>
-  </xacro:if>
   <xacro:if value="$(arg kinect_enabled)">
     <xacro:sensor_arch prefix="" parent="top_plate_link">
@@ -170,4 +161,46 @@
   </gazebo>
   <!-- Optional custom includes. -->
-  <xacro:include filename="$(arg urdf_extras)" />
+  <link name="umbc_structure_mesh">
+    <visual>
+      <geometry>
+        <mesh filename="package://umbc_husky/meshes/UMBC_structure.STL"/>
+      </geometry>
+      <material name="charcoal">
+        <color rgba="0.2 0.2 0.2 1"/>
+      </material>
+    </visual>
+  </link>
+  <joint name="top_plate_to_umbc_tower_mesh" type="fixed">
+    <parent link="top_plate_link"/>
+    <child link="umbc_structure_mesh"/>
+    <origin xyz="-0.06 0 0.007" rpy="0 0 0" />
+  </joint>
+  <link name="upper_top_plate">
+    <visual>
+      <geometry>
+        <mesh filename="package://husky_description/meshes/top_plate.dae"/>
+      </geometry>
+    </visual>
+  </link>
+  <joint name="top_plate_to_upper_top_plate" type="fixed">
+    <parent link="top_plate_link"/>
+    <child link="upper_top_plate"/>
+    <origin xyz="0.0 0.0 0.307" rpy="0 0 0" />
+  </joint>
+  <!-- Create a fixed joint to connect the Kinect2 to the rest of the robot -->
+  <link name="kinect2_link" />
+  <joint name="top_plate_to_kinect2" type="fixed">
+    <parent link="top_plate_link"/>
+    <child link="kinect2_link"/>
+    <origin xyz="-0.30 0.0 0.59" rpy="-1.57079633 0 -1.57079633" />
+  </joint>
+  <!-- Create a fixed joint to connect the Jaco to the rest of the robot -->
+  <xacro:include filename="$(find kinova_description)/urdf/j2n6s300.xacro" />
+  <link name="right_arm_link"/>
+  <joint name="top_plate_to_right_arm" type="fixed">
+    <parent link="top_plate_link"/>
+    <child link="right_arm_link"/>
+    <origin xyz="0.21 -0.197 0.315" rpy="0 0 1.57079633" />
+  </joint>
+  <xacro:j2n6s300 base_parent="right_arm_link" prefix="j2n6s300" />
 </robot>

Commit message: added navigation with rtab, update urdf and launch files to allow for arm to be enabled/disabled, still need to get arm control working, and manage navigation with the arm moving infron of sensor

File: urdf/umbc_husky.urdf.xacro (robot description, xacro)
@@ -22,8 +22,7 @@
 -->
 <robot name="husky" xmlns:xacro="http://www.ros.org/wiki/xacro">
-  <xacro:arg name="laser_enabled" default="false" />
   <xacro:arg name="laser_xyz" default="$(optenv HUSKY_LMS1XX_XYZ 0.2206 0.0 0.00635)" />
   <xacro:arg name="laser_rpy" default="$(optenv HUSKY_LMS1XX_RPY 0.0 0.0 0.0)" />
-  <xacro:arg name="kinect_enabled" default="true" />
+  <xacro:arg name="arm_enabled" default="true" />
   <xacro:arg name="kinect_xyz" default="$(optenv HUSKY_KINECT_XYZ 0 0 0)" />
   <xacro:arg name="kinect_rpy" default="$(optenv HUSKY_KINECT_RPY 0 0.18 3.14)" />
@@ -115,15 +114,13 @@
   </xacro:husky_wheel>
   <xacro:husky_decorate />
-  <xacro:if value="$(arg kinect_enabled)">
-    <xacro:sensor_arch prefix="" parent="top_plate_link">
-      <origin xyz="-0.35 0 0.51" rpy="0 0 -3.14"/>
-    </xacro:sensor_arch>
-    <joint name="kinect_frame_joint" type="fixed">
-      <origin xyz="$(arg kinect_xyz)" rpy="$(arg kinect_rpy)" />
-      <parent link="sensor_arch_mount_link"/>
-      <child link="camera_link"/>
-    </joint>
-    <xacro:kinect_camera prefix="camera" robot_namespace="$(arg robot_namespace)"/>
-  </xacro:if>
+  <xacro:sensor_arch prefix="" parent="top_plate_link">
+    <origin xyz="-0.35 0 0.51" rpy="0 0 -3.14"/>
+  </xacro:sensor_arch>
+  <joint name="kinect_frame_joint" type="fixed">
+    <origin xyz="$(arg kinect_xyz)" rpy="$(arg kinect_rpy)" />
+    <parent link="sensor_arch_mount_link"/>
+    <child link="camera_link"/>
+  </joint>
+  <xacro:kinect_camera prefix="camera" robot_namespace="$(arg robot_namespace)"/>
   <gazebo>
     <plugin name="gazebo_ros_control" filename="libgazebo_ros_control.so">
@@ -195,12 +192,14 @@
     <origin xyz="-0.30 0.0 0.59" rpy="-1.57079633 0 -1.57079633" />
   </joint>
-  <!-- Create a fixed joint to connect the Jaco to the rest of the robot -->
-  <xacro:include filename="$(find kinova_description)/urdf/j2n6s300.xacro" />
-  <link name="right_arm_link"/>
-  <joint name="top_plate_to_right_arm" type="fixed">
-    <parent link="top_plate_link"/>
-    <child link="right_arm_link"/>
-    <origin xyz="0.21 -0.197 0.315" rpy="0 0 1.57079633" />
-  </joint>
-  <xacro:j2n6s300 base_parent="right_arm_link" prefix="j2n6s300" />
+  <xacro:if value="$(arg arm_enabled)">
+    <!-- Create a fixed joint to connect the Jaco to the rest of the robot -->
+    <xacro:include filename="$(find kinova_description)/urdf/j2n6s300.xacro" />
+    <link name="right_arm_link"/>
+    <joint name="top_plate_to_right_arm" type="fixed">
+      <parent link="top_plate_link"/>
+      <child link="right_arm_link"/>
+      <origin xyz="0.21 -0.197 0.315" rpy="0 0 1.57079633" />
+    </joint>
+    <xacro:j2n6s300 base_parent="right_arm_link" prefix="j2n6s300" />
+  </xacro:if >
 </robot>

Commit message: Urdf working with both jaco arm and husky controllers in gazebo, added simple script to point the arm at things given a point

File: urdf/umbc_husky.urdf.xacro (robot description, xacro)
@@ -125,5 +125,4 @@
   <gazebo>
     <plugin name="gazebo_ros_control" filename="libgazebo_ros_control.so">
-      <robotNamespace>$(arg robot_namespace)</robotNamespace>
     </plugin>
   </gazebo>
@@ -199,5 +198,6 @@
       <parent link="top_plate_link"/>
       <child link="right_arm_link"/>
-      <origin xyz="0.21 -0.197 0.315" rpy="0 0 1.57079633" />
+      <!-- org <origin xyz="0.21 -0.197 0.315" rpy="0 0 1.57079633" /> -->
+      <origin xyz="0.21 -0.197 0.315" rpy="0 0 0" />
     </joint>
     <xacro:j2n6s300 base_parent="right_arm_link" prefix="j2n6s300" />
