Commit message: added collison to arm parts of husky urdf

File: umbc_husky/urdf/umbc_husky_full.urdf (robot description, URDF)
Before this commit: robot husky, 36 links, 35 joints
Links:
- link camera_link: geometry collision box size=0.07 0.3 0.09
- link j2n6s300_link_1: geometry collision mesh filename=package://kinova_description/meshes/ring_big.dae; collision mesh filename=package://kinova_description/meshes/shoulder.dae
- link j2n6s300_link_2: geometry collision mesh filename=package://kinova_description/meshes/arm.dae; collision mesh filename=package://kinova_description/meshes/ring_big.dae
- link j2n6s300_link_3: geometry collision mesh filename=package://kinova_description/meshes/forearm.dae; collision mesh filename=package://kinova_description/meshes/ring_big.dae
- link j2n6s300_link_4: geometry collision mesh filename=package://kinova_description/meshes/ring_small.dae; collision mesh filename=package://kinova_description/meshes/wrist.dae
- link j2n6s300_link_5: geometry collision mesh filename=package://kinova_description/meshes/ring_small.dae; collision mesh filename=package://kinova_description/meshes/wrist.dae
- link upper_top_plate: geometry collision mesh filename=package://husky_description/meshes/top_plate.dae; visual mesh filename=package://husky_description/meshes/top_plate.dae

Commit message: Update umbc_husky_full.urdf

File: umbc_husky/urdf/umbc_husky_full.urdf (robot description, URDF)
Before this commit: robot husky, 36 links, 35 joints
Links:
- link camera_link: geometry 
- link j2n6s300_link_6: geometry collision mesh filename=package://kinova_description/meshes/hand_3finger.dae; collision mesh filename=package://kinova_description/meshes/ring_small.dae
Joints:
- joint j2n6s300_joint_finger_1: origin xyz=0.00279 0.03126 -0.11467 rpy=-1.570796327 .649262481663582 1.35961148639407 -> xyz=0.00279 0.03126 -0.11467 rpy=-1.7047873384941834 0.6476144647144773 1.67317415161155
- joint top_plate_to_kinect2: origin xyz=-0.30 0.0 0.59 rpy=-1.57079633 0 -1.57079633 -> xyz=-0.30 -0.1 0.57 rpy=-1.57079633 0 -1.57079633
- joint top_plate_to_right_arm: origin xyz=0.21 -0.197 0.315 rpy=0 0 0 -> xyz=0.22 -0.197 0.315 rpy=0 0 0

Commit message: Revert "Update umbc_husky_full.urdf"
This reverts commit da378dc273be4798297e671fdd211f11dc3626fe.

File: umbc_husky/urdf/umbc_husky_full.urdf (robot description, URDF)
Before this commit: robot husky, 36 links, 35 joints
Links:
- link camera_link: geometry collision box size=0.07 0.3 0.09
- link j2n6s300_link_6: geometry collision mesh filename=package://kinova_description/meshes/hand_3finger.dae; visual mesh filename=package://kinova_description/meshes/hand_3finger.dae
Joints:
- joint j2n6s300_joint_finger_1: origin xyz=0.00279 0.03126 -0.11467 rpy=-1.7047873384941834 0.6476144647144773 1.67317415161155 -> xyz=0.00279 0.03126 -0.11467 rpy=-1.570796327 .649262481663582 1.35961148639407
- joint top_plate_to_kinect2: origin xyz=-0.30 -0.1 0.57 rpy=-1.57079633 0 -1.57079633 -> xyz=-0.30 0.0 0.59 rpy=-1.57079633 0 -1.57079633
- joint top_plate_to_right_arm: origin xyz=0.22 -0.197 0.315 rpy=0 0 0 -> xyz=0.21 -0.197 0.315 rpy=0 0 0
